File: kicad/DisplayAdapter.sch (KiCad schematic (older format))
At the start: 4 parts

Commit message: Revision 3
Parts:
- removed Q?: IRLML2502, Micro3, symbol FieldDevice_R2:IRLML2502
- added Q?: Q_NMOS_GSD, symbol Device:Q_NMOS_GSD
- added R? (x2): 20Ω, symbol Device:R
- added U?: EA_DOGS104x-A, symbol FieldDevice_R2:EA_DOGS104x-A
- R?: value R -> 10kΩ
Connections:
- net GND: now also C?.2, C?.2, R?.2, R?.1, R?.1, U?.12 (IM1), U?.14 (Vss), U?.18 (CS), U?.19 (SA0~)
- net SCL: now also U?.17 (SLCK~)
- net SDA: now also U?.15 (SOD), U?.16 (SID)
- net Vbb: now also C?.1, Q?.3 (D), U?.13 (Vdd)
- net BACKLIGHT: now reaches R?.1
- net BACKLIGHT: now also Q?.1 (G)
- net Vout: now reaches C?.1
- net Vout: now also U?.11 (Vout)
- new net: Q?.2 (S), U?.1 (A1/AGR/AEWR), U?.10 (A2/NC/CW)
- new net: R?.2, U?.2 (C1/CR/CR)
- new net: R?.2, U?.9 (C2/CG/CE)
- new net ~RESET: U?.20 (~RESET)
Other:
- note added: "EA DOGS104-A\nEA LED36X28-A Amber Backlight"
- moved on the sheet: C?, R?
